Commit message: 更新urdf

File: src/piper_description/urdf/piper_no_gripper_description.xacro (robot description, xacro)
@@ -14,31 +14,17 @@
     <inertial>
       <origin
-        xyz="-0.00973928490005031 1.83127089286717E-06 0.0410140167677137"
-        rpy="0 0 0" />
-      <mass
-        value="0.0001" />
-      <inertia
-        ixx="0.000226592553127906"
-        ixy="-7.33974356968615E-08"
-        ixz="2.13221970218122E-06"
-        iyy="0.000269447877479622"
-        iyz="8.15167478682596E-09"
-        izz="0.000222318286704" />
-    </inertial>
-    <visual>
-      <origin
-        xyz="0 0 0"
-        rpy="1.5708 0 -1.5708" />
-      <geometry>
-        <mesh
-          filename="package://piper_description/meshes/base_link.dae" />
-      </geometry>
-      <material
-        name="">
-        <color
-          rgba="0.792156862745098 0.819607843137255 0.933333333333333 1" />
-      </material>
-    </visual>
-    <collision>
+        xyz="-0.00473641164191482 2.56829134630247E-05 0.041451518036016"
+        rpy="0 0 0" />
+      <mass
+        value="0.333893486740112" />
+      <inertia
+        ixx="0.000254953479570424"
+        ixy="2.06931238580746E-07"
+        ixz="7.30912474718368E-06"
+        iyy="0.00027202099920186"
+        iyz="2.65131745382267E-07"
+        izz="0.000276534627629623" />
+    </inertial>
+    <visual>
       <origin
         xyz="0 0 0"
@@ -48,4 +34,18 @@
           filename="package://piper_description/meshes/base_link.STL" />
       </geometry>
+      <material
+        name="">
+        <color
+          rgba="0.792156862745098 0.819607843137255 0.933333333333333 1" />
+      </material>
+    </visual>
+    <collision>
+      <origin
+        xyz="0 0 0"
+        rpy="0 0 0" />
+      <geometry>
+        <mesh
+          filename="package://piper_description/meshes/base_link.STL" />
+      </geometry>
     </collision>
   </link>
@@ -54,31 +54,17 @@
     <inertial>
       <origin
-        xyz="0.00131676031927021 0.000310288842008365 -0.00922874512303438"
-        rpy="0 0 0" />
-      <mass
-        value="0.0001" />
-      <inertia
-        ixx="7.76684558296782E-05"
-        ixy="1.09084650459916E-07"
-        ixz="-1.97480532432411E-06"
-        iyy="9.24967780161546E-05"
-        iyz="9.91284646834672E-07"
-        izz="8.24589062407806E-05" />
-    </inertial>
-    <visual>
-      <origin
-        xyz="0 0 0"
-        rpy="1.5708 0 0" />
-      <geometry>
-        <mesh
-          filename="package://piper_description/meshes/link1.dae" />
-      </geometry>
-      <material
-        name="">
-        <color
-          rgba="0.792156862745098 0.819607843137255 0.933333333333333 1" />
-      </material>
-    </visual>
-    <collision>
+        xyz="0.000121504734057468 0.000104632162460536 -0.00438597309559853"
+        rpy="0 0 0" />
+      <mass
+        value="0.215052383265765" />
+      <inertia
+        ixx="0.000109639007860341"
+        ixy="2.50631260865109E-07"
+        ixz="-1.89352789149844E-07"
+        iyy="9.95612262461418E-05"
+        iyz="1.00634716976093E-08"
+        izz="0.000116363910317385" />
+    </inertial>
+    <visual>
       <origin
         xyz="0 0 0"
@@ -88,4 +74,18 @@
           filename="package://piper_description/meshes/link1.STL" />
       </geometry>
+      <material
+        name="">
+        <color
+          rgba="0.792156862745098 0.819607843137255 0.933333333333333 1" />
+      </material>
+    </visual>
+    <collision>
+      <origin
+        xyz="0 0 0"
+        rpy="0 0 0" />
+      <geometry>
+        <mesh
+          filename="package://piper_description/meshes/link1.STL" />
+      </geometry>
     </collision>
   </link>
@@ -95,5 +95,5 @@
     <origin
       xyz="0 0 0.123"
-      rpy="0 0 -1.5708" />
+      rpy="0 0 0" />
     <parent
       link="base_link" />
@@ -104,7 +104,7 @@
     <limit
       lower="-2.618"
-      upper="2.618"
-      effort="100"
-      velocity="3" />
+      upper="2.168"
+      effort="100"
+      velocity="5" />
   </joint>
   <link
@@ -112,31 +112,17 @@
     <inertial>
       <origin
-        xyz="0.147615838821413 -0.0174259998251394 0.00175952516190707"
-        rpy="0 0 0" />
-      <mass
-        value="0.0001" />
-      <inertia
-        ixx="0.000150112628108228"
-        ixy="8.58974959950769E-05"
-        ixz="-1.07428153464284E-06"
-        iyy="0.00172585302855383"
-        iyz="-9.93704792239676E-07"
-        izz="0.00177445942914759" />
-    </inertial>
-    <visual>
-      <origin
-        xyz="0 0 0"
-        rpy="0 1.5708 -0.0873" />
-      <geometry>
-        <mesh
-          filename="package://piper_description/meshes/link2.dae" />
-      </geometry>
-      <material
-        name="">
-        <color
-          rgba="0.792156862745098 0.819607843137255 0.933333333333333 1" />
-      </material>
-    </visual>
-    <collision>
+        xyz="0.198666145229743 -0.010926924140076 0.00142121714502687"
+        rpy="0 0 0" />
+      <mass
+        value="0.463914239236335" />
+      <inertia
+        ixx="0.000214137415059993"
+        ixy="7.26120579340088E-05"
+        ixz="-9.88224861011274E-07"
+        iyy="0.00100030277518254"
+        iyz="-1.32818212212246E-06"
+        izz="0.00104417184176783" />
+    </inertial>
+    <visual>
       <origin
         xyz="0 0 0"
@@ -146,4 +132,18 @@
           filename="package://piper_description/meshes/link2.STL" />
       </geometry>
+      <material
+        name="">
+        <color
+          rgba="0.792156862745098 0.819607843137255 0.933333333333333 1" />
+      </material>
+    </visual>
+    <collision>
+      <origin
+        xyz="0 0 0"
+        rpy="0 0 0" />
+      <geometry>
+        <mesh
+          filename="package://piper_description/meshes/link2.STL" />
+      </geometry>
     </collision>
   </link>
@@ -153,5 +153,5 @@
     <origin
       xyz="0 0 0"
-      rpy="1.5708 -0.10095 -1.5708" />
+      rpy="1.5708 -0.10095 -3.1416" />
     <parent
       link="link1" />
@@ -164,5 +164,5 @@
       upper="3.14"
       effort="100"
-      velocity="3" />
+      velocity="5" />
   </joint>
   <link
@@ -170,31 +170,17 @@
     <inertial>
       <origin
-        xyz="0.0156727239770991 0.104466514402189 0.000508486576356504"
-        rpy="0 0 0" />
-      <mass
-        value="0.0001" />
-      <inertia
-        ixx="0.00022168634302318"
-        ixy="-7.57426147001315E-06"
-        ixz="-6.36999759250492E-07"
-        iyy="0.000100859159512329"
-        iyz="-8.16199264787698E-07"
-        izz="0.000241839306422341" />
-    </inertial>
-    <visual>
-      <origin
-        xyz="0 0 0"
-        rpy="1.4835 1.5708 0" />
-      <geometry>
-        <mesh
-          filename="package://piper_description/meshes/link3.dae" />
-      </geometry>
-      <material
-        name="">
-        <color
-          rgba="0.792156862745098 0.819607843137255 0.933333333333333 1" />
-      </material>
-    </visual>
-    <collision>
+        xyz="-0.0202737662122021 -0.133914995944595 -0.000458682652737356"
+        rpy="0 0 0" />
+      <mass
+        value="0.219942452993132" />
+      <inertia
+        ixx="0.00018953849076141"
+        ixy="-8.05719205057736E-06"
+        ixz="5.10255053956334E-07"
+        iyy="7.1424497082494E-05"
+        iyz="8.89044974368937E-07"
+        izz="0.000201212938725775" />
+    </inertial>
+    <visual>
       <origin
         xyz="0 0 0"
@@ -204,4 +190,18 @@
           filename="package://piper_description/meshes/link3.STL" />
       </geometry>
+      <material
+        name="">
+        <color
+          rgba="0.792156862745098 0.819607843137255 0.933333333333333 1" />
+      </material>
+    </visual>
+    <collision>
+      <origin
+        xyz="0 0 0"
+        rpy="0 0 0" />
+      <geometry>
+        <mesh
+          filename="package://piper_description/meshes/link3.STL" />
+      </geometry>
     </collision>
   </link>
@@ -211,5 +211,5 @@
     <origin
       xyz="0.28503 0 0"
-      rpy="0 0 1.3826" />
+      rpy="0 0 -1.759" />
     <parent
       link="link2" />
@@ -222,5 +222,5 @@
       upper="0"
       effort="100"
-      velocity="3" />
+      velocity="5" />
   </joint>
   <link
@@ -228,31 +228,17 @@
     <inertial>
       <origin
-        xyz="0.000276464622388145 -0.00102803669324856 -0.00472830700561582"
-        rpy="0 0 0" />
-      <mass
-        value="0.0001" />
-      <inertia
-        ixx="3.82011730423392E-05"
-        ixy="-4.92358350916331E-08"
-        ixz="4.89589432971791E-08"
-        iyy="4.87048555222583E-05"
-        iyz="6.70802942501353E-08"
-        izz="4.10592077565539E-05" />
-    </inertial>
-    <visual>
-      <origin
-        xyz="0 0 0"
-        rpy="1.48 0 1.5708" />
-      <geometry>
-        <mesh
-          filename="package://piper_description/meshes/link4.dae" />
-      </geometry>
-      <material
-        name="">
-        <color
-          rgba="0.792156862745098 0.819607843137255 0.933333333333333 1" />
-      </material>
-    </visual>
-    <collision>
+        xyz="-9.66635791618542E-05 0.000876064475651083 -0.00496880904640868"
+        rpy="0 0 0" />
+      <mass
+        value="0.131814339939458" />
+      <inertia
+        ixx="3.96965423235175E-05"
+        ixy="-2.32268338444837E-08"
+        ixz="-1.14702090783249E-07"
+        iyy="5.13319789853892E-05"
+        iyz="9.92852686264567E-08"
+        izz="4.14768131680711E-05" />
+    </inertial>
+    <visual>
       <origin
         xyz="0 0 0"
@@ -262,4 +248,18 @@
           filename="package://piper_description/meshes/link4.STL" />
       </geometry>
+      <material
+        name="">
+        <color
+          rgba="0.792156862745098 0.819607843137255 0.933333333333333 1" />
+      </material>
+    </visual>
+    <collision>
+      <origin
+        xyz="0 0 0"
+        rpy="0 0 0" />
+      <geometry>
+        <mesh
+          filename="package://piper_description/meshes/link4.STL" />
+      </geometry>
     </collision>
   </link>
@@ -268,6 +268,6 @@
     type="revolute">
     <origin
-      xyz="0.021984 0.25075 0"
-      rpy="-1.5708 0 0" />
+      xyz="-0.021984 -0.25075 0"
+      rpy="1.5708 0 0" />
     <parent
       link="link3" />
@@ -280,5 +280,5 @@
       upper="1.832"
       effort="100"
-      velocity="3" />
+      velocity="5" />
   </joint>
   <link
@@ -286,31 +286,17 @@
     <inertial>
       <origin
-        xyz="8.82262433637704E-05 0.0566829014808264 -0.00196119720482555"
-        rpy="0 0 0" />
-      <mass
-        value="0.0001" />
-      <inertia
-        ixx="4.39644313661978E-05"
-        ixy="-3.59259686449865E-08"
-        ixz="-1.89747741592145E-08"
-        iyy="5.6317392095077E-05"
-        iyz="-2.1540716689678E-07"
-        izz="4.88713664675246E-05" />
-    </inertial>
-    <visual>
-      <origin
-        xyz="0 0 0"
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
Commit message: update urdf joint limit

File: src/piper_description/urdf/piper_description.urdf (robot description, URDF)
Before this commit: robot piper_description, 10 links, 9 joints
Joints:
- joint joint3: limit lower=-2.697 upper=0 effort=100 velocity=5 -> lower=-2.967 upper=0 effort=100 velocity=5
- joint joint4: limit lower=-1.832 upper=1.832 effort=100 velocity=5 -> lower=-1.745 upper=1.745 effort=100 velocity=5

File: src/piper_description/urdf/piper_no_gripper_description.urdf (robot description, URDF)
Before this commit: robot piper_description, 7 links, 6 joints
Joints:
- joint joint3: limit lower=-2.697 upper=0 effort=100 velocity=5 -> lower=-2.967 upper=0 effort=100 velocity=5
- joint joint4: limit lower=-1.832 upper=1.832 effort=100 velocity=5 -> lower=-1.745 upper=1.745 effort=100 velocity=5
